File: EsquematicoCorregido.brd (EAGLE design)
At the start: 70.9 x 80 mm, 45 parts, among them IC1 OPA991TIDCKR, IC10 MCP73831T-2ACI_OT, IC2 AD8226ARZ-RL, IC3 OPA991TIDCKR, IC4 ESP32-S3-WROOM-1-N16R8, IC5 OPA991TIDCKR, IC6 MAX30102EFD+T, IC7 LP38692MP-3.3_NOPB, IC8 LP38692MP-1.8_NOPB, IC9 REF2033AIDDCT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

Commit message: pcb
Routing:
- net VSS: track 64.4 -> 84.7 mm, vias 2 -> 4
Changed lines of the file:
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@@
 <wire x1="14.097" y1="25.273" x2="17.145" y2="25.273" width="0.4064" layer="1"/>
 <wire x1="18.481" y1="26.609" x2="18.481" y2="28.702" width="0.4064" layer="1"/>
-<wire x1="17.145" y1="25.273" x2="18.481" y2="26.609" width="0.4064" layer="1"/>
+<wire x1="17.145" y1="25.273" x2="17.526" y2="25.654" width="0.4064" layer="1"/>
+<wire x1="17.526" y1="25.654" x2="18.481" y2="26.609" width="0.4064" layer="1"/>
 <wire x1="19.324" y1="20" x2="14.925" y2="20" width="0.4064" layer="1"/>
 <wire x1="14.925" y1="20" x2="14.097" y2="20.828" width="0.4064" layer="1"/>
@@
 <wire x1="11.43" y1="22.86" x2="11.43" y2="25.273" width="0.4064" layer="1"/>
 <wire x1="9.144" y1="2.667" x2="10.16" y2="3.683" width="0.4064" layer="16"/>
-<wire x1="19.324" y1="20" x2="12.872" y2="13.335" width="0" layer="19" extent="1-1"/>
+<wire x1="12.872" y1="13.335" x2="15.494" y2="13.335" width="0.4064" layer="1"/>
+<via x="15.494" y="13.335" extent="1-16" drill="0.35"/>
+<wire x1="15.494" y1="13.335" x2="18.288" y2="13.335" width="0.4064" layer="16"/>
+<wire x1="19.812" y1="14.859" x2="19.812" y2="25.019" width="0.4064" layer="16"/>
+<via x="19.812" y="25.019" extent="1-16" drill="0.35"/>
+<wire x1="19.812" y1="25.019" x2="19.177" y2="25.654" width="0.4064" layer="1"/>
+<wire x1="19.177" y1="25.654" x2="17.526" y2="25.654" width="0.4064" layer="1"/>
+<wire x1="18.288" y1="13.335" x2="19.812" y2="14.859" width="0.4064" layer="16"/>
 </signal>
 <signal name="INA">

Commit message: avance PCB
Routing:
- net D-: track 0.00 -> 68.3 mm, vias 0 -> 2
- net D+: track 0.00 -> 2.77 mm
Changed lines of the file:
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@@
 <contactref element="J3" pad="A7"/>
 <contactref element="J3" pad="B7"/>
-<wire x1="61.48" y1="6.894" x2="48.4" y2="57.33" width="0" layer="19" extent="1-1"/>
-<wire x1="62.48" y1="6.894" x2="61.48" y2="6.894" width="0" layer="19" extent="1-1"/>
+<wire x1="61.48" y1="6.894" x2="61.48" y2="8.775" width="0.3048" layer="1"/>
+<wire x1="61.48" y1="8.775" x2="61.722" y2="9.017" width="0.3048" layer="1"/>
+<wire x1="61.722" y1="9.017" x2="62.103" y2="9.017" width="0.3048" layer="1"/>
+<wire x1="62.103" y1="9.017" x2="62.48" y2="8.64" width="0.3048" layer="1"/>
+<wire x1="62.48" y1="8.64" x2="62.48" y2="6.894" width="0.3048" layer="1"/>
+<wire x1="61.48" y1="6.894" x2="61.48" y2="5.473" width="0.3048" layer="1"/>
+<wire x1="61.48" y1="5.473" x2="61.468" y2="5.461" width="0.3048" layer="1"/>
+<via x="61.468" y="5.461" extent="1-16" drill="0.35"/>
+<wire x1="61.468" y1="5.461" x2="61.468" y2="5.4929875" width="0.3048" layer="16"/>
+<wire x1="61.468" y1="5.4929875" x2="44.45" y2="22.5109875" width="0.3048" layer="16"/>
+<wire x1="44.45" y1="22.5109875" x2="44.45" y2="55.88" width="0.3048" layer="16"/>
+<via x="44.45" y="55.88" extent="1-16" drill="0.35"/>
+<wire x1="44.45" y1="55.88" x2="45.9" y2="57.33" width="0.3048" layer="1"/>
+<wire x1="45.9" y1="57.33" x2="48.4" y2="57.33" width="0.3048" layer="1"/>
 </signal>
 <signal name="D+">
@@
 <contactref element="J3" pad="A6"/>
 <contactref element="J3" pad="B6"/>
+<wire x1="61.98" y1="6.894" x2="61.98" y2="6.1" width="0.254" layer="1"/>
+<wire x1="61.98" y1="6.1" x2="61.976" y2="6.096" width="0.254" layer="1"/>
+<wire x1="61.976" y1="6.096" x2="62.1665" y2="5.9055" width="0.254" layer="1"/>
+<wire x1="62.1665" y1="5.9055" x2="62.8015" y2="5.9055" width="0.254" layer="1"/>
+<wire x1="62.98" y1="6.084" x2="62.98" y2="6.894" width="0.254" layer="1"/>
+<wire x1="62.8015" y1="5.9055" x2="62.98" y2="6.084" width="0.254" layer="1"/>
 <wire x1="61.98" y1="6.894" x2="48.4" y2="56.06" width="0" layer="19" extent="1-1"/>
-<wire x1="62.98" y1="6.894" x2="61.98" y2="6.894" width="0" layer="19" extent="1-1"/>
 </signal>
 <signal name="N$18">

Commit message: Pistas del conector micro usb-c
Routing:
- net D+: track 2.77 -> 73.9 mm, vias 0 -> 2
Changed lines of the file:
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@@
 <wire x1="61.48" y1="5.473" x2="61.468" y2="5.461" width="0.3048" layer="1"/>
 <via x="61.468" y="5.461" extent="1-16" drill="0.35"/>
-<wire x1="61.468" y1="5.461" x2="61.468" y2="5.4929875" width="0.3048" layer="16"/>
-<wire x1="61.468" y1="5.4929875" x2="44.45" y2="22.5109875" width="0.3048" layer="16"/>
-<wire x1="44.45" y1="22.5109875" x2="44.45" y2="55.88" width="0.3048" layer="16"/>
+<wire x1="61.468" y1="5.461" x2="61.468" y2="6.3819875" width="0.3048" layer="16"/>
+<wire x1="61.468" y1="6.3819875" x2="44.45" y2="23.3999875" width="0.3048" layer="16"/>
+<wire x1="44.45" y1="23.3999875" x2="44.45" y2="55.88" width="0.3048" layer="16"/>
 <via x="44.45" y="55.88" extent="1-16" drill="0.35"/>
 <wire x1="44.45" y1="55.88" x2="45.9" y2="57.33" width="0.3048" layer="1"/>
@@
 <contactref element="J3" pad="A6"/>
 <contactref element="J3" pad="B6"/>
-<wire x1="61.98" y1="6.894" x2="61.98" y2="6.1" width="0.254" layer="1"/>
-<wire x1="61.98" y1="6.1" x2="61.976" y2="6.096" width="0.254" layer="1"/>
+<wire x1="61.98" y1="6.1" x2="61.98" y2="6.894" width="0.254" layer="1"/>
+<wire x1="61.976" y1="6.096" x2="61.98" y2="6.1" width="0.254" layer="1"/>
 <wire x1="61.976" y1="6.096" x2="62.1665" y2="5.9055" width="0.254" layer="1"/>
-<wire x1="62.1665" y1="5.9055" x2="62.8015" y2="5.9055" width="0.254" layer="1"/>
-<wire x1="62.98" y1="6.084" x2="62.98" y2="6.894" width="0.254" layer="1"/>
+<wire x1="62.1665" y1="5.9055" x2="62.23" y2="5.9055" width="0.254" layer="1"/>
+<wire x1="62.8015" y1="5.9055" x2="62.23" y2="5.9055" width="0.254" layer="1"/>
+<wire x1="62.98" y1="6.084" x2="62.98" y2="6.35" width="0.254" layer="1"/>
+<wire x1="62.98" y1="6.894" x2="62.98" y2="6.35" width="0.254" layer="1"/>
 <wire x1="62.8015" y1="5.9055" x2="62.98" y2="6.084" width="0.254" layer="1"/>
-<wire x1="61.98" y1="6.894" x2="48.4" y2="56.06" width="0" layer="19" extent="1-1"/>
+<wire x1="62.98" y1="6.35" x2="62.992" y2="6.338" width="0.3048" layer="1"/>
+<wire x1="62.992" y1="6.338" x2="62.992" y2="5.08" width="0.3048" layer="1"/>
+<via x="62.992" y="5.08" extent="1-16" drill="0.35"/>
+<wire x1="62.992" y1="5.08" x2="63.627" y2="4.445" width="0.3048" layer="16"/>
+<wire x1="64.2920125" y1="4.445" x2="64.6114125" y2="4.1256" width="0.3048" layer="16"/>
+<wire x1="64.6114125" y1="4.1256" x2="68.041125" y2="4.1256" width="0.3048" layer="16"/>
+<wire x1="68.041125" y1="4.1256" x2="69.630671875" y2="5.715146875" width="0.3048" layer="16"/>
+<wire x1="69.630671875" y1="5.715146875" x2="69.630671875" y2="8.093328125" width="0.3048" layer="16"/>
+<wire x1="46.101" y1="31.623" x2="46.101" y2="54.61" width="0.3048" layer="16"/>
+<via x="46.101" y="54.61" extent="1-16" drill="0.35"/>
+<wire x1="46.101" y1="54.61" x2="46.101" y2="55.753" width="0.3048" layer="1"/>
+<wire x1="46.408" y1="56.06" x2="48.4" y2="56.06" width="0.3048" layer="1"/>
+<wire x1="63.627" y1="4.445" x2="64.2920125" y2="4.445" width="0.3048" layer="16"/>
+<wire x1="69.630671875" y1="8.093328125" x2="46.101" y2="31.623" width="0.3048" layer="16"/>
+<wire x1="46.101" y1="55.753" x2="46.408" y2="56.06" width="0.3048" layer="1"/>
 </signal>
 <signal name="N$18">
