File: EsquematicoCorregido.brd (EAGLE design)
At the start: 70.9 x 80 mm, 45 parts, among them IC1 OPA991TIDCKR, IC10 MCP73831T-2ACI_OT, IC2 AD8226ARZ-RL, IC3 OPA991TIDCKR, IC4 ESP32-S3-WROOM-1-N16R8, IC5 OPA991TIDCKR, IC6 MAX30102EFD+T, IC7 LP38692MP-3.3_NOPB, IC8 LP38692MP-1.8_NOPB, IC9 REF2033AIDDCT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

Commit message: ultimo avance
Parts:
- moved C11 25.2 mm to (45.7, 75.7), turned to 270 degrees
- moved RST 1.78 mm to (37.6, 73.8)
- moved R13 1.02 mm to (31.8, 71.0)
- moved J2 0.89 mm to (2.54, 5.46)
- moved R12 0.51 mm to (32.3, 58.8)
Connections:
- removed net 3V3: C11.2
- net +3V3: now also C11.2
Routing:
- net +3V3: track 159.2 -> 264.4 mm, vias 4 -> 6
- net OUT-ADC: track 7.80 -> 43.0 mm, vias 0 -> 2
- net COMM: track 15.4 -> 39.1 mm, vias 0 -> 2
- net BATT+: track 11.7 -> 31.4 mm, vias 0 -> 2
- net EN: track 17.4 -> 19.1 mm
- net INA-: track 33.3 -> 34.2 mm
- net INA+: track 2.94 -> 3.83 mm
- net OUTFILT: track 17.2 -> 17.7 mm
- net IO0: track 42.3 -> 41.7 mm

Commit message: avances
Routing:
- net GND: vias 26 -> 28
Changed lines of the file:
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@@
 <via x="6.35" y="48.26" extent="1-16" drill="0.35"/>
 <via x="12.7" y="45.72" extent="1-16" drill="0.35"/>
-<wire x1="57.05" y1="66.25" x2="65.9" y2="72.57" width="0" layer="19" extent="1-1"/>
-<wire x1="55.65" y1="66.25" x2="57.05" y2="66.25" width="0" layer="19" extent="1-1"/>
-<wire x1="57.05" y1="64.85" x2="57.05" y2="66.25" width="0" layer="19" extent="1-1"/>
-<wire x1="54.25" y1="66.25" x2="55.65" y2="66.25" width="0" layer="19" extent="1-1"/>
-<wire x1="57.05" y1="63.45" x2="57.05" y2="64.85" width="0" layer="19" extent="1-1"/>
-<wire x1="54.25" y1="64.85" x2="54.25" y2="66.25" width="0" layer="19" extent="1-1"/>
-<wire x1="55.65" y1="64.85" x2="55.65" y2="66.25" width="0" layer="19" extent="1-1"/>
-<wire x1="55.65" y1="63.45" x2="57.05" y2="63.45" width="0" layer="19" extent="1-1"/>
-<wire x1="54.25" y1="63.45" x2="54.25" y2="64.85" width="0" layer="19" extent="1-1"/>
-<wire x1="48.4" y1="72.57" x2="54.25" y2="66.25" width="0" layer="19" extent="1-1"/>
-<wire x1="45.72" y1="76.642" x2="48.4" y2="72.57" width="0" layer="19" extent="1-1"/>
-<wire x1="35.1" y1="61.54" x2="45.72" y2="76.642" width="0" layer="19" extent="1-1"/>
-<wire x1="34.592" y1="75.637" x2="45.72" y2="76.642" width="0" layer="19" extent="1-1"/>
-<wire x1="15.24" y1="50.8" x2="35.1" y2="61.54" width="0" layer="19" extent="1-1"/>
-<wire x1="12.7" y1="45.72" x2="15.24" y2="50.8" width="0" layer="19" extent="1-1"/>
-<wire x1="6.35" y1="48.26" x2="12.7" y2="45.72" width="0" layer="19" extent="1-1"/>
-<wire x1="18.1" y1="39.37" x2="12.7" y2="45.72" width="0" layer="19" extent="1-1"/>
-<wire x1="5.4" y1="39.37" x2="6.35" y2="48.26" width="0" layer="19" extent="1-1"/>
-<wire x1="29.53" y1="39.37" x2="18.1" y2="39.37" width="0" layer="19" extent="1-1"/>
-<wire x1="35.24" y1="35.56" x2="29.53" y2="39.37" width="0" layer="19" extent="1-1"/>
-<wire x1="36.83" y1="35.56" x2="35.24" y2="35.56" width="0" layer="19" extent="1-1"/>
-<wire x1="36.83" y1="33.02" x2="36.83" y2="35.56" width="0" layer="19" extent="1-1"/>
-<wire x1="41.91" y1="35.56" x2="36.83" y2="35.56" width="0" layer="19" extent="1-1"/>
-<wire x1="41.91" y1="33.02" x2="41.91" y2="35.56" width="0" layer="19" extent="1-1"/>
-<wire x1="44.516" y1="31.369" x2="41.91" y2="33.02" width="0" layer="19" extent="1-1"/>
-<wire x1="35.56" y1="25.4" x2="36.83" y2="33.02" width="0" layer="19" extent="1-1"/>
-<wire x1="30.48" y1="26.67" x2="35.56" y2="25.4" width="0" layer="19" extent="1-1"/>
-<wire x1="29.611" y1="17.399" x2="30.48" y2="26.67" width="0" layer="19" extent="1-1"/>
-<wire x1="25.527" y1="16.957" x2="29.611" y2="17.399" width="0" layer="19" extent="1-1"/>
-<wire x1="26.241" y1="2.832" x2="28.591" y2="8.382" width="0" layer="19" extent="1-1"/>
-<wire x1="19.324" y1="19.05" x2="25.527" y2="16.957" width="0" layer="19" extent="1-1"/>
-<wire x1="32.941" y1="2.832" x2="26.241" y2="2.832" width="0" layer="19" extent="1-1"/>
-<wire x1="35.179" y1="13.274" x2="28.514" y2="12.319" width="0" layer="19" extent="1-1"/>
-<wire x1="12.872" y1="12.065" x2="19.324" y2="19.05" width="0" layer="19" extent="1-1"/>
-<wire x1="8.636" y1="20.193" x2="12.872" y2="12.065" width="0" layer="19" extent="1-1"/>
-<wire x1="8.128" y1="21.082" x2="8.636" y2="20.193" width="0" layer="19" extent="1-1"/>
-<wire x1="9.271" y1="21.082" x2="8.636" y2="20.193" width="0" layer="19" extent="1-1"/>
-<wire x1="7.493" y1="20.193" x2="8.128" y2="21.082" width="0" layer="19" extent="1-1"/>
-<wire x1="6.985" y1="21.082" x2="7.493" y2="20.193" width="0" layer="19" extent="1-1"/>
-<wire x1="6.35" y1="20.193" x2="6.985" y2="21.082" width="0" layer="19" extent="1-1"/>
-<wire x1="5.842" y1="21.082" x2="6.35" y2="20.193" width="0" layer="19" extent="1-1"/>
-<wire x1="5.207" y1="20.193" x2="5.842" y2="21.082" width="0" layer="19" extent="1-1"/>
-<wire x1="4.699" y1="21.082" x2="5.207" y2="20.193" width="0" layer="19" extent="1-1"/>
-<wire x1="8.128" y1="22.86" x2="8.128" y2="21.082" width="0" layer="19" extent="1-1"/>
-<wire x1="7.62" y1="23.749" x2="8.128" y2="22.86" width="0" layer="19" extent="1-1"/>
-<wire x1="8.763" y1="23.749" x2="8.128" y2="22.86" width="0" layer="19" extent="1-1"/>
-<wire x1="9.271" y1="22.86" x2="8.763" y2="23.749" width="0" layer="19" extent="1-1"/>
-<wire x1="6.985" y1="22.86" x2="7.62" y2="23.749" width="0" layer="19" extent="1-1"/>
-<wire x1="6.477" y1="23.749" x2="6.985" y2="22.86" width="0" layer="19" extent="1-1"/>
-<wire x1="5.842" y1="22.86" x2="6.477" y2="23.749" width="0" layer="19" extent="1-1"/>
-<wire x1="5.334" y1="23.749" x2="5.842" y2="22.86" width="0" layer="19" extent="1-1"/>
-<wire x1="4.699" y1="22.86" x2="5.334" y2="23.749" width="0" layer="19" extent="1-1"/>
-<wire x1="50.802" y1="16.51" x2="44.516" y2="27.686" width="0" layer="19" extent="1-1"/>
-<wire x1="57.135" y1="6.244" x2="50.802" y2="16.51" width="0" layer="19" extent="1-1"/>
-<wire x1="59.03" y1="6.894" x2="57.135" y2="6.244" width="0" layer="19" extent="1-1"/>
-<wire x1="57.135" y1="2.319" x2="57.135" y2="6.244" width="0" layer="19" extent="1-1"/>
-<wire x1="65.43" y1="6.894" x2="59.03" y2="6.894" width="0" layer="19" extent="1-1"/>
-<wire x1="67.325" y1="6.244" x2="65.43" y2="6.894" width="0" layer="19" extent="1-1"/>
-<wire x1="67.325" y1="2.319" x2="67.325" y2="6.244" width="0" layer="19" extent="1-1"/>
-<wire x1="65.024" y1="13.142" x2="65.43" y2="6.894" width="0" layer="19" extent="1-1"/>
-<wire x1="68.072" y1="13.142" x2="65.024" y2="13.142" width="0" layer="19" extent="1-1"/>
-<wire x1="63.502" y1="16.637" x2="65.024" y2="13.142" width="0" layer="19" extent="1-1"/>
+<via x="53.34" y="16.51" extent="1-16" drill="0.35"/>
+<via x="54.61" y="6.35" extent="1-16" drill="0.35"/>
 <wire x1="63.03" y1="39.44" x2="44.516" y2="31.369" width="0" layer="19" extent="1-1"/>
+<wire x1="34.592" y1="75.637" x2="35.1" y2="61.54" width="0" layer="19" extent="1-1"/>
+<wire x1="45.72" y1="76.642" x2="34.592" y2="75.637" width="0" layer="19" extent="1-1"/>
 </signal>
 <signal name="N$4">
@@
 <wire x1="59.944" y1="9.271" x2="59.8474" y2="9.1744" width="0.4064" layer="1"/>
 <wire x1="59.8474" y1="9.1744" x2="59.8474" y2="8.128" width="0.4064" layer="1"/>
-<wire x1="59.8474" y1="8.128" x2="59.8474" y2="6.93143125" width="0.4064" layer="1"/>
+<wire x1="59.8474" y1="6.93143125" x2="59.8474" y2="8.128" width="0.4064" layer="1"/>
 <wire x1="38.608" y1="12.7" x2="41.275" y2="12.7" width="0.4064" layer="1"/>
 <wire x1="41.275" y1="12.7" x2="42.418" y2="11.557" width="0.4064" layer="1"/>
@@
 <wire x1="42.418" y1="9.398" x2="43.053" y2="8.763" width="0.4064" layer="1"/>
 <wire x1="44.958" y1="8.763" x2="45.466" y2="8.255" width="0.4064" layer="1"/>
-<wire x1="45.466" y1="8.255" x2="45.466" y2="7.62" width="0.4064" layer="1"/>
-<wire x1="45.466" y1="7.62" x2="45.466" y2="7.239" width="0.4064" layer="1"/>
+<wire x1="45.466" y1="8.255" x2="45.466" y2="7.239" width="0.4064" layer="1"/>
 <wire x1="45.466" y1="7.239" x2="45.466" y2="4.719" width="0.3048" layer="1"/>
 <wire x1="45.466" y1="4.719" x2="45.514" y2="4.671" width="0.3048" layer="1"/>
@@
 <wire x1="59.2124" y1="8.763" x2="59.8474" y2="8.128" width="0.4064" layer="1"/>
 <wire x1="46.101" y1="8.763" x2="59.2124" y2="8.763" width="0.4064" layer="1"/>
-<wire x1="59.8474" y1="6.93143125" x2="59.83" y2="6.894" width="0" layer="19" extent="1-1"/>
+<wire x1="59.83" y1="6.894" x2="59.83" y2="6.91403125" width="0.3048" layer="1"/>
+<wire x1="59.83" y1="6.91403125" x2="59.8474" y2="6.93143125" width="0.3048" layer="1"/>
 </signal>
 <signal name="N$1">
