File: EsquematicoCorregido.sch (EAGLE design)
At the start: 45 parts, among them IC1 OPA991TIDCKR, IC10 MCP73831T-2ACI_OT, IC2 AD8226ARZ-RL, IC3 OPA991TIDCKR, IC4 ESP32-S3-WROOM-1-N16R8, IC5 OPA991TIDCKR, IC6 MAX30102EFD+T, IC7 LP38692MP-3.3_NOPB, IC8 LP38692MP-1.8_NOPB, IC9 REF2033AIDDCT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

Commit message: modificaciones PCB
Connections:
- net VDD renamed +1V8
- removed net N$21: OLED.1
- net GND: now also OLED.1
- net OUTFILT: no longer IC4.IO12
Changed lines of the file:
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@@
 <part name="SUPPLY11" library="supply2" library_urn="urn:adsk.eagle:library:372" deviceset="VSS" device=""/>
 <part name="SUPPLY12" library="supply2" library_urn="urn:adsk.eagle:library:372" deviceset="GND" device=""/>
-<part name="VDD1" library="supply1" library_urn="urn:adsk.eagle:library:371" deviceset="VDD" device=""/>
-<part name="VDD2" library="supply1" library_urn="urn:adsk.eagle:library:371" deviceset="VDD" device=""/>
 <part name="SUPPLY1" library="supply2" library_urn="urn:adsk.eagle:library:372" deviceset="VSS" device=""/>
 <part name="SUPPLY3" library="supply2" library_urn="urn:adsk.eagle:library:372" deviceset="VSS" device=""/>
@@
 <part name="+3V6" library="supply1" library_urn="urn:adsk.eagle:library:371" deviceset="+3V3" device=""/>
 <part name="+3V8" library="supply1" library_urn="urn:adsk.eagle:library:371" deviceset="+3V3" device=""/>
+<part name="+3V13" library="supply1" library_urn="urn:adsk.eagle:library:371" deviceset="+3V3" device=""/>
+<part name="P+1" library="supply1" library_urn="urn:adsk.eagle:library:371" deviceset="VCC" device="" value="+1V8"/>
 </parts>
 <sheets>
@@
 <attribute name="VALUE" x="262.255" y="217.805" size="1.778" layer="96"/>
 </instance>
-<instance part="VDD1" gate="G$1" x="5.08" y="165.1" smashed="yes">
-<attribute name="VALUE" x="2.54" y="162.56" size="1.778" layer="96" rot="R90"/>
-</instance>
-<instance part="VDD2" gate="G$1" x="182.88" y="137.16" smashed="yes">
-<attribute name="VALUE" x="184.912" y="140.716" size="1.778" layer="96" rot="R180"/>
-</instance>
 <instance part="SUPPLY1" gate="G$1" x="134.62" y="195.58" smashed="yes">
 <attribute name="VALUE" x="132.715" y="190.881" size="1.778" layer="96"/>
@@
 <instance part="+3V8" gate="G$1" x="68.58" y="91.44" smashed="yes">
 <attribute name="VALUE" x="66.04" y="86.36" size="1.778" layer="96" rot="R90"/>
+</instance>
+<instance part="+3V13" gate="G$1" x="182.88" y="137.16" smashed="yes"/>
+<instance part="P+1" gate="VCC" x="5.08" y="167.64" smashed="yes">
+<attribute name="VALUE" x="2.54" y="165.1" size="1.778" layer="96" rot="R90"/>
 </instance>
 </instances>
@@
 <wire x1="246.38" y1="60.96" x2="241.3" y2="60.96" width="0.1524" layer="91"/>
 </segment>
+<segment>
+<pinref part="OLED" gate="1" pin="1"/>
+<wire x1="5.08" y1="93.98" x2="12.7" y2="93.98" width="0.1524" layer="91"/>
+<pinref part="SUPPLY25" gate="GND" pin="GND"/>
+<wire x1="12.7" y1="88.9" x2="12.7" y2="93.98" width="0.1524" layer="91"/>
+</segment>
 </net>
 <net name="N$4" class="0">
@@
 <net name="OUTFILT" class="0">
 <segment>
-<pinref part="IC4" gate="G$1" pin="IO12"/>
-<wire x1="279.4" y1="177.8" x2="274.32" y2="177.8" width="0.1524" layer="91"/>
-<label x="269.24" y="177.8" size="1.778" layer="95"/>
-</segment>
-<segment>
 <wire x1="220.98" y1="228.6" x2="210.82" y2="228.6" width="0.1524" layer="91" style="longdash"/>
 <label x="210.82" y="228.6" size="1.778" layer="95"/>
@@
 </segment>
 </net>
-<net name="VDD" class="0">
-<segment>
-<pinref part="VDD1" gate="G$1" pin="VDD"/>
-<pinref part="IC8" gate="G$1" pin="OUT"/>
-<wire x1="5.08" y1="162.56" x2="5.08" y2="157.48" width="0.1524" layer="91"/>
-<wire x1="5.08" y1="157.48" x2="12.7" y2="157.48" width="0.1524" layer="91"/>
-</segment>
-<segment>
-<pinref part="IC6" gate="G$1" pin="VDD"/>
-<wire x1="137.16" y1="137.16" x2="144.78" y2="137.16" width="0.1524" layer="91"/>
-<wire x1="144.78" y1="137.16" x2="144.78" y2="132.08" width="0.1524" layer="91"/>
-<wire x1="172.72" y1="132.08" x2="172.72" y2="134.62" width="0.1524" layer="91"/>
-<wire x1="157.48" y1="134.62" x2="157.48" y2="132.08" width="0.1524" layer="91"/>
-<wire x1="157.48" y1="132.08" x2="172.72" y2="132.08" width="0.1524" layer="91"/>
-<wire x1="144.78" y1="132.08" x2="157.48" y2="132.08" width="0.1524" layer="91"/>
-<junction x="157.48" y="132.08"/>
-<pinref part="VDD2" gate="G$1" pin="VDD"/>
-<wire x1="182.88" y1="134.62" x2="182.88" y2="132.08" width="0.1524" layer="91"/>
-<wire x1="182.88" y1="132.08" x2="172.72" y2="132.08" width="0.1524" layer="91"/>
-<junction x="172.72" y="132.08"/>
-<pinref part="C8" gate="G$1" pin="1"/>
-<wire x1="157.48" y1="137.16" x2="157.48" y2="134.62" width="0.1524" layer="91" style="longdash"/>
-<pinref part="C5" gate="G$1" pin="1"/>
-<wire x1="172.72" y1="137.16" x2="172.72" y2="134.62" width="0.1524" layer="91" style="longdash"/>
-</segment>
-</net>
 <net name="OUT-ADC" class="0">
 <segment>
@@
 </segment>
 </net>
-<net name="N$21" class="0">
-<segment>
-<pinref part="OLED" gate="1" pin="1"/>
-<wire x1="5.08" y1="93.98" x2="12.7" y2="93.98" width="0.1524" layer="91"/>
-<wire x1="12.7" y1="93.98" x2="12.7" y2="88.9" width="0.1524" layer="91"/>
-<pinref part="SUPPLY25" gate="GND" pin="GND"/>
-</segment>
-</net>
 <net name="N$1" class="0">
 <segment>
@@
 </segment>
 </net>
+<net name="+1V8" class="0">
+<segment>
+<pinref part="IC6" gate="G$1" pin="VDD"/>
+<wire x1="137.16" y1="137.16" x2="144.78" y2="137.16" width="0.1524" layer="91"/>
+<wire x1="144.78" y1="137.16" x2="144.78" y2="132.08" width="0.1524" layer="91"/>
+<wire x1="172.72" y1="132.08" x2="172.72" y2="134.62" width="0.1524" layer="91"/>
+<wire x1="157.48" y1="134.62" x2="157.48" y2="132.08" width="0.1524" layer="91"/>
+<wire x1="157.48" y1="132.08" x2="172.72" y2="132.08" width="0.1524" layer="91"/>
+<wire x1="144.78" y1="132.08" x2="157.48" y2="132.08" width="0.1524" layer="91"/>
+<junction x="157.48" y="132.08"/>
+<wire x1="182.88" y1="134.62" x2="182.88" y2="132.08" width="0.1524" layer="91"/>
+<wire x1="182.88" y1="132.08" x2="172.72" y2="132.08" width="0.1524" layer="91"/>
+<junction x="172.72" y="132.08"/>
+<pinref part="C8" gate="G$1" pin="1"/>
+<wire x1="157.48" y1="137.16" x2="157.48" y2="134.62" width="0.1524" layer="91" style="longdash"/>
+<pinref part="C5" gate="G$1" pin="1"/>
+<wire x1="172.72" y1="137.16" x2="172.72" y2="134.62" width="0.1524" layer="91" style="longdash"/>
+<pinref part="+3V13" gate="G$1" pin="+3V3"/>
+<label x="185.42" y="128.778" size="1.778" layer="95" rot="R90"/>
+</segment>
+<segment>
+<pinref part="IC8" gate="G$1" pin="OUT"/>
+<wire x1="5.08" y1="157.48" x2="12.7" y2="157.48" width="0.1524" layer="91"/>
+<wire x1="5.08" y1="165.1" x2="5.08" y2="157.48" width="0.1524" layer="91"/>
+<pinref part="P+1" gate="VCC" pin="VCC"/>
+<label x="2.54" y="165.1" size="1.778" layer="95" rot="R90"/>
+</segment>
+</net>

Commit message: ultimo avance
Connections:
- removed net 3V3: C11.2
- net +3V3: now also C11.2
Changed lines of the file:
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@@
 <part name="+3V13" library="supply1" library_urn="urn:adsk.eagle:library:371" deviceset="+3V3" device=""/>
 <part name="P+1" library="supply1" library_urn="urn:adsk.eagle:library:371" deviceset="VCC" device="" value="+1V8"/>
+<part name="+3V14" library="supply1" library_urn="urn:adsk.eagle:library:371" deviceset="+3V3" device=""/>
 </parts>
 <sheets>
@@
 <attribute name="VALUE" x="2.54" y="165.1" size="1.778" layer="96" rot="R90"/>
 </instance>
+<instance part="+3V14" gate="G$1" x="177.8" y="81.28" smashed="yes" rot="R270">
+<attribute name="VALUE" x="172.72" y="83.82" size="1.778" layer="96"/>
+</instance>
 </instances>
 <busses>
@@
 <wire x1="68.58" y1="88.9" x2="68.58" y2="86.36" width="0.1524" layer="91" style="longdash"/>
 </segment>
+<segment>
+<pinref part="C11" gate="G$1" pin="2"/>
+<wire x1="165.1" y1="81.28" x2="175.26" y2="81.28" width="0.1524" layer="91"/>
+<pinref part="+3V14" gate="G$1" pin="+3V3"/>
+</segment>
 </net>
 <net name="N$6" class="0">
@@
 </segment>
 </net>
-<net name="3V3" class="0">
-<segment>
-<wire x1="167.64" y1="81.28" x2="177.8" y2="81.28" width="0.1524" layer="91" style="longdash"/>
-<label x="175.26" y="81.28" size="1.778" layer="95" rot="R180"/>
-<pinref part="C11" gate="G$1" pin="2"/>
-<wire x1="165.1" y1="81.28" x2="167.64" y2="81.28" width="0.1524" layer="91"/>
-</segment>
-</net>
